File: rfidAntenna38x41.kicad_pcb (KiCad board)
At the start: 2 copper layers, 40 x 43 mm, 16 parts, among them J1 Conn_01x03_Pin

Commit message: updates
Parts:
- added J2: Conn_01x02_Pin, rfidAntenna38x41:PinHeader_1x02_P2.54mm_Vertical, F.Cu at (163.0, 111.0)
- moved R2 1.01 mm to (160.2, 112.6)
- moved R1 1.01 mm to (155.3, 112.6)
- moved R3 0.99 mm to (168.4, 112.5)
- moved R4 0.99 mm to (173.3, 112.5)
Routing:
- net Net-(J2-Pin_1): track 24.2 -> 33.4 mm
