File: rfidAntenna38x41.kicad_sch (KiCad schematic)
At the start: 16 parts, among them J1 Conn_01x03_Pin

Commit message: updates
Parts:
- added J2: Conn_01x02_Pin, rfidAntenna38x41:PinHeader_1x02_P2.54mm_Vertical, symbol Connector:Conn_01x02_Pin
Connections:
- net at L1.1, L1.2, R1.1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: now also J2.1 (Pin_1), J2.2 (Pin_2)
Changed lines of the file:
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@@
+    (stroke (width 0) (type default))
+  )
+  (wire (pts (xy 180.975 85.09) (xy 180.975 87.63))
     (stroke (width 0) (type default))
   )
@@
     (stroke (width 0) (type default))
   )
+  (wire (pts (xy 174.625 85.09) (xy 180.975 85.09))
+    (stroke (width 0) (type default))
+  )
   (wire (pts (xy 102.235 91.44) (xy 102.235 99.06))
     (stroke (width 0) (type default))
@@
     (stroke (width 0) (type default))
   )
+  (wire (pts (xy 180.975 92.71) (xy 174.625 92.71))
+    (stroke (width 0) (type default))
+  )
   (wire (pts (xy 136.525 88.9) (xy 136.525 91.44))
     (stroke (width 0) (type default))
@@
   )
   (wire (pts (xy 161.925 78.74) (xy 161.925 74.93))
+    (stroke (width 0) (type default))
+  )
+  (wire (pts (xy 180.975 90.17) (xy 180.975 92.71))
     (stroke (width 0) (type default))
   )
@@
         )
       )
+    )
+  )
+  (symbol (lib_id "Connector:Conn_01x02_Pin") (at 186.055 87.63 0) (mirror y) (unit 1)
+    (in_bom yes) (on_board yes) (dnp no)
+    (property "Reference" "J2" (at 186.7662 89.5437 0)
+      (effects (font (size 1.27 1.27)) (justify right))
+    )
+    (property "Value" "Conn_01x02_Pin" (at 186.7662 87.6227 0)
+      (effects (font (size 1.27 1.27)) (justify right) hide)
+    )
+    (property "Footprint" "rfidAntenna38x41:PinHeader_1x02_P2.54mm_Vertical" (at 186.055 87.63 0)
+      (effects (font (size 1.27 1.27)) hide)
+    )
+    (property "Datasheet" "~" (at 186.055 87.63 0)
+      (effects (font (size 1.27 1.27)) hide)
+    )
+    (pin "1")
+    (pin "2")
+    (instances
+      (project "rfidAntenna38x41"
+        (path "/8278437e-f37f-44e4-8f76-ad3ae44bdaed"
+          (reference "J2") (unit 1)
+        )
+      )
